File: Hardware/placa_manutencao_preventiva/placa_manutencao_preventiva.sch (KiCad schematic (older format))
At the start: 20 parts, among them J1 ENT_DIGITAL, J2 Power, J3 TESTE_TENSAO, J4 BAT_EXT_JST_1.25mm, J5 BAT_HELTEC_CONN, J6 MPU6050, J7 BMP180, J8 Renewable energy, Q2 FQP30N06L, U1 Heltec_Wifi_LoRa_V1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

Commit message: Vers 1.1: Devolopment area
Parts:
- added C4, C5, C6, C7: 0.1uF, Capacitor_THT:C_Disc_D5.1mm_W3.2mm_P5.00mm, symbol Device:C
- added J12, J13, J14, J15, J16, J17, J18, J19, J20, J21, J22, J23, J24, J25: Conn_01x01, Connector_Pin:Pin_D0.9mm_L10.0mm_W2.4mm_FlatFork, symbol Connector_Generic:Conn_01x01
- C1: value 0.33uF -> 10uF
- C2: footprint Capacitor_THT:CP_Radial_D5.0mm_P2.00mm -> Capacitor_THT:C_Disc_D5.1mm_W3.2mm_P5.00mm; symbol Device:CP1 -> Device:C
- Q2: symbol FQP30N06L:FQP30N06L -> placa_manutencao_preventiva-rescue:FQP30N06L-FQP30N06L
- U1: symbol heltec_wifi_lora_v1:Heltec_Wifi_LoRa_V1 -> placa_manutencao_preventiva-rescue:Heltec_Wifi_LoRa_V1-heltec_wifi_lora_v1
Connections:
- net +3V3: now also C4.1, C5.1
- net +5V: now also C6.1, C7.1
- net ADC_BAT: now also J20.1 (Pin_1)
- net GND: now also C4.2, C5.2, C6.2, C7.2
- net I2C_SCL: now also J14.1 (Pin_1)
- net I2C_SDA: now also J16.1 (Pin_1)
- net at U1.12 (LORA_CS/V_SPI_CLK/GPIO18): now also J12.1 (Pin_1)
- net at U1.13 (LORA_SCK/V_SPI_CS0/GPIO5): now also J13.1 (Pin_1)
- net at U1.15 (TOUCH2/HSPI_WP/ADC2_2/GPIO2): now also J15.1 (Pin_1)
- net at U1.17 (U2_TX/GPIO17): now also J17.1 (Pin_1)
- net at U1.18 (OLED_RST/U2_RX/GPIO16): now also J18.1 (Pin_1)
- net at U1.19 (V_SPI_HD/SDA/GPIO21): now also J19.1 (Pin_1)
- net at U1.21 (TOUCH5/ADC2_5/GPIO12): now also J21.1 (Pin_1)
- net at U1.22 (LORA_RST/TOUCH6/ADC2_6/GPIO14): now also J22.1 (Pin_1)
- net at U1.23 (LORA_MOSI/TOUCH7/ADC2_7/GPIO27): now also J23.1 (Pin_1)
- net at U1.24 (LORA_DIO0/DAC1/ADC2_9/GPIO26): now also J24.1 (Pin_1)
- net at U1.25 (LED/DAC2/ADC2_8/GPIO25): now also J25.1 (Pin_1)
Other:
- moved on the sheet: J2, J3, J4, J5, J6, J7, R4, R5
